File: shinyu/_autosave-shinyu.kicad_pcb (KiCad board)
At the start: 2 copper layers, 36 x 46 mm, 12 parts, among them IC1 GL823K, J1 USB_C_Receptacle_USB2.0_16P, J2 SD_Card_Receptacle, U1 AP2112K

Commit message: last com 4 tonight
kicking ts bucket. finished tracing with 0 errors and opened my 3d viewer to see i had the wrong footprint for my usb c plug 🥰 that no its actuallyt amazing! its exactly what i wanted! so im restarting TOMORROW aint NO WAY im doing this tonight
Parts:
- J1: footprint Connector_USB:USB_C_Plug_ShenzhenJingTuoJin_918-118A2021Y40002_Vertical -> Connector_USB:USB_C_Receptacle_GCT_USB4085
- U1: value AP2112K -> AP2112K-3.3
- moved C6 8.83 mm to (146.2, 89.0)
- moved C5 6.20 mm to (160.8, 96.1)
- moved J1 4.79 mm to (167.2, 94.9), turned to 90 degrees
- moved R2 4.46 mm to (159.7, 93.1)
- moved C4 4.31 mm to (146.1, 95.7)
- moved U1 1.55 mm to (165.4, 99.8)
Routing:
- net /VBUS_5V: track 39.8 -> 7.41 mm
- net /3V3: track 26.7 -> 0.00 mm
- net /CLK: track 24.8 -> 0.00 mm
- net /D1: track 23.7 -> 0.00 mm, vias 2 -> 0
- net /D0: track 22.8 -> 0.00 mm, vias 2 -> 0
- net GND: track 0.00 -> 18.6 mm
- net /CC2: track 0.00 -> 13.2 mm, vias 0 -> 2
- net /USB_DP: track 14.1 -> 2.02 mm, vias 0 -> 1
- net /CC1: track 9.22 -> 0.00 mm
- net /USB_DM: track 14.1 -> 13.0 mm, vias 2 -> 0
- net /D2: track 34.6 -> 35.4 mm
