File: shinyu/shinyu.kicad_sch (KiCad schematic)
At the start: 12 parts, among them IC1 GL823K, J1 USB_C_Receptacle_USB2.0_16P, J2 SD_Card_Receptacle, U1 AP2112K-3.3

Commit message: last com 4 tonight
kicking ts bucket. finished tracing with 0 errors and opened my 3d viewer to see i had the wrong footprint for my usb c plug 🥰 that no its actuallyt amazing! its exactly what i wanted! so im restarting TOMORROW aint NO WAY im doing this tonight
Parts:
- J1: footprint Connector_USB:USB_C_Plug_ShenzhenJingTuoJin_918-118A2021Y40002_Vertical -> Connector_USB:USB_C_Receptacle_GCT_USB4085
Changed lines of the file:
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@@
 			)
 		)
-		(property "Footprint" "Connector_USB:USB_C_Plug_ShenzhenJingTuoJin_918-118A2021Y40002_Vertical"
+		(property "Footprint" "Connector_USB:USB_C_Receptacle_GCT_USB4085"
 			(at 63.5 60.96 0)
 			(effects
