File: a-side/a-side.kicad_pcb (KiCad board)
At the start: 2 copper layers, 95 x 60 mm, 37 parts, among them IC1 GL823K, IC2 GL823K, J1 Conn_01x06, J2 503500-0993, J3 503500-0993, J4 USB_A, J5 USB_A, U1 AMS1117CD-3.3, U2 SRV05-4, Y1 Crystal

Commit message: ???? short ahh
cant sleep so decided to do a 5 min work sesh , added 2 leds for the sd card readers ohh my god chat i literally cant fall asleep its 4 am 😭
Parts:
- added D1: LED, LED_SMD:LED_0805_2012Metric_Pad1.15x1.40mm_HandSolder, F.Cu at (23.1, 85.2)
- added D2: LED, LED_SMD:LED_0805_2012Metric_Pad1.15x1.40mm_HandSolder, F.Cu at (23.1, 88.2)
- added R7: 330R, Resistor_SMD:R_0805_2012Metric, F.Cu at (27.7, 85.2)
- added R8: 330R, Resistor_SMD:R_0805_2012Metric, F.Cu at (27.7, 88.1)
- C2: value 22uF -> 10uF
- J1: value Conn_01x06 -> Conn_01x04; footprint Connector_PinHeader_2.54mm:PinHeader_1x06_P2.54mm_Vertical -> Connector_PinHeader_2.54mm:PinHeader_1x04_P2.54mm_Vertical
- moved J1 26.2 mm to (47.6, 82.9)
Connections:
- IC1 pad 12: unconnected-(IC1-LED-Pad12) -> Net-(IC1-LED)
- IC2 pad 12: unconnected-(IC2-LED-Pad12) -> Net-(IC2-LED)
