File: a-side/a-side.kicad_pcb (KiCad board)
At the start: 2 copper layers, 95 x 55 mm, 40 parts, among them IC1 GL823K, IC2 GL823K, J2 USB_C_Receptacle_USB2.0_14P, J4 USB_A, J5 USB_A, U1 AMS1117CD-3.3, U2 SRV05-4, Y1 Crystal

Commit message: fixing..
schematic... fixing orientation on stuffs... fixing footprints again... fixing...
Parts:
- added J6: SD_Card_Receptacle, Connector_Card:SD_Card_Device_16mm_SlotDepth, F.Cu at (107.0, 121.0)
- added J7: SD_Card_Receptacle, Connector_Card:SD_Card_Device_16mm_SlotDepth, F.Cu at (144.6, 121.0)
- added R11: 10k, Resistor_SMD:R_0805_2012Metric, F.Cu at (100.2, 100.8)
- added R12: 10k, Resistor_SMD:R_0805_2012Metric, F.Cu at (103.1, 100.8)
- added R13: 10k, Resistor_SMD:R_0805_2012Metric, F.Cu at (106.0, 100.8)
- added R14: 10k, Resistor_SMD:R_0805_2012Metric, F.Cu at (109.0, 100.8)
- added R15: 10k, Resistor_SMD:R_0805_2012Metric, F.Cu at (112.0, 100.8)
- added R16: 10k, Resistor_SMD:R_0805_2012Metric, F.Cu at (137.9, 101.8)
- added R17: 10k, Resistor_SMD:R_0805_2012Metric, F.Cu at (140.8, 101.8)
- added R18: 10k, Resistor_SMD:R_0805_2012Metric, F.Cu at (143.8, 101.8)
- added R19: 10k, Resistor_SMD:R_0805_2012Metric, F.Cu at (146.8, 101.8)
- added R20: 10k, Resistor_SMD:R_0805_2012Metric, F.Cu at (149.7, 101.8)
Connections:
- C18 pad 1: GND -> +3.3V
- C18 pad 2: +3.3V -> GND
- C3 pad 1: VBUS -> GND
- C3 pad 2: GND -> VBUS
- D1 pad 1: Net-(D1-K) -> GND
- D1 pad 2: GND -> Net-(D1-A)
- D2 pad 1: Net-(D2-K) -> GND
- D2 pad 2: GND -> Net-(D2-A)
- R7 pad 2: Net-(D1-K) -> Net-(D1-A)
- R8 pad 2: Net-(D2-K) -> Net-(D2-A)
