File: a-side/a-side.kicad_sch (KiCad schematic)
At the start: 37 parts, among them IC1 GL823K, IC2 GL823K, J1 Conn_01x06, J2 503500-0993, J3 503500-0993, J4 USB_A, J5 USB_A, U1 AMS1117CD-3.3, U2 SRV05-4, Y1 Crystal

Commit message: ???? short ahh
cant sleep so decided to do a 5 min work sesh , added 2 leds for the sd card readers ohh my god chat i literally cant fall asleep its 4 am 😭
Parts:
- removed J1: Conn_01x06, Connector_PinHeader_2.54mm:PinHeader_1x06_P2.54mm_Vertical, symbol Connector_Generic:Conn_01x06
- added D1, D2: LED, LED_SMD:LED_0805_2012Metric_Pad1.15x1.40mm_HandSolder, symbol Device:LED
- added J1: Conn_01x04, Connector_PinHeader_2.54mm:PinHeader_1x04_P2.54mm_Vertical, symbol Connector_Generic:Conn_01x04
- C2: value 22uF -> 10uF
- R7, R8: value 5.1kR -> 330R
Connections:
- net CC1 is gone; now on an unnamed net: R7.1
- net CC2 is gone; now on an unnamed net: R8.1
- net GND: now also D1.2 (A), D2.2 (A), J1.2 (Pin_2)
- net USB_DM: now also J1.4 (Pin_4)
- net USB_DP: now also J1.3 (Pin_3)
- net VBUS: now also J1.1 (Pin_1)
- net at R7.2: now also D1.1 (K)
- net at R8.2: now also D2.1 (K)
- no-connect marks 25 -> 23
