File: a-side/a-side.kicad_sch (KiCad schematic)
At the start: 39 parts, among them IC1 GL823K, IC2 GL823K, J2 USB_C_Receptacle_USB2.0_14P, J4 USB_A, J5 USB_A, J6 SD_Card_Receptacle, J7 SD_Card_Receptacle, U1 AMS1117CD-3.3, U2 SRV05-4, Y1 Crystal

Commit message: last commie of the day!
fixed major issues earlier, rn just fixing some decoupling caps here and there heh i mean all in a days work what can i say
Parts:
- added C19: 100nF, symbol Device:C
- added R10, R9: 5.1k, symbol Device:R
Connections:
- net +3.3V: now also J6.4 (VDD), J7.4 (VDD)
- net GND: now also C19.2, R10.2, R9.2
- net VBUS: now also U2.5 (VP), C19.1
- net at J2.A5 (CC1): now also R9.1
- net at J2.B5 (CC2): now also R10.1
- net SD1_PWR: no longer names the net of IC1.8 (PMOS)
- net SD1_PWR: no longer J6.4 (VDD)
- net SD2_PWR: no longer names the net of IC2.8 (PMOS)
- net SD2_PWR: no longer J7.4 (VDD)
- no-connect marks 15 -> 14
Other:
- note added: "IF ITS A CAPACITOR with a pwr label on one side and NOT directly connected to the pin it's porbably for decoupling !!!!!!!!"
- note removed: "footprinting...."
- note removed: "still cant find the standard sd card receptacle for some reaosn"
- moved on the sheet: C12, C13, C14, C15, C16, C17, D1, D2, IC1, IC2, J2, J6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
