File: a-side/a-side.kicad_sch (KiCad schematic)
At the start: 56 parts, among them IC3 GL823K, IC4 GL823K, J1 USB_A, J2 SD_Card_Receptacle, J3 USB_A, J4 USB_C_Receptacle_USB2.0_14P, J5 SD_Card_Receptacle, SW1 SW_Push, U1 SRV05-4, U2 SRV05-4, Y1 12MHz

Commit message: getting deep into routing
just gonna commit rn coz im a little locked in but uhh yea schema done i think, footprints all found
Parts:
- removed Y1: 12MHz, Crystal:Crystal_SMD_3225-4Pin_3.2x2.5mm_HandSoldering, symbol Device:Crystal
- added Y2: Crystal_GND24, Crystal:Crystal_SMD_3225-4Pin_3.2x2.5mm, symbol Device:Crystal_GND24
Connections:
- net GND: now also Y2.2 (G), Y2.4 (G)
- net at C1.2, GL850G2.6 (X1): now also Y2.3
- net at C2.1, GL850G2.7 (X2): now also Y2.1

Commit message: DOME
done done done DONE 0 errors 108982 warnings who gaf im done
Parts:
- removed J1, J3: USB_A, Connector_USB:USB_A_Connfly_DS1098_Horizontal, symbol Connector:USB_A
- removed J2, J5: SD_Card_Receptacle, Connector_Card:SD_Kyocera_145638009511859+, symbol Connector:SD_Card_Receptacle
- removed J4: USB_C_Receptacle_USB2.0_14P, Connector_USB:USB_C_Receptacle_HRO_TYPE-C-31-M-12, symbol Connector:USB_C_Receptacle_USB2.0_14P
- removed R9: 5.1k, Resistor_SMD:R_0805_2012Metric, symbol Device:R
- added Card1, Card2: SD-106M, easyeda2kicad:SD-SMD_SD-106M, symbol easyeda2kicad:SD-106M
- added R23: 5.1k, Resistor_SMD:R_0805_2012Metric, symbol Device:R
- added USB1, USB2: AF 90° WJDG, easyeda2kicad:USB-A-TH_AF-WJDG, symbol easyeda2kicad:AF90°WJDG
- added USB3: TYPE-C 16PIN 2MD, easyeda2kicad:USB-C-SMD_TYPE-C-16PIN-2MD-073, symbol easyeda2kicad:TYPE-C16PIN2MD
Connections:
- net +3V3 is gone; now on net +3.3V: R11.1, R12.1, R13.1, R14.1, R15.1, R16.1, R17.1, R18.1, R19.1, R2.2, R20.1, R5.2, R6.2
- net GND: now also Card1.11 (WP), Card1.12 (SHELL), Card1.13 (SHELL), Card1.3 (VSS1), Card1.6 (VSS2), Card2.11 (WP), Card2.12 (SHELL), Card2.13 (SHELL), Card2.3 (VSS1), Card2.6 (VSS2), R23.1, USB1.4 (GND), USB1.5 (SHLD), USB2.4 (GND), USB2.5 (SHLD), USB3.13 (EH), USB3.14 (EH), USB3.A1B12 (GND), USB3.B1A12 (GND); no longer IC3.10 (5V), IC4.10 (5V)
- net SD1_CLK: now also Card1.5 (CLK)
- net SD1_CMD: now also Card1.2 (CMD)
- net SD1_D0: now also Card1.7 (DAT0)
- net SD1_D1: now also Card1.8 (DAT1)
- net SD1_D2: now also Card1.9 (DAT2)
- net SD1_D3: now also Card1.1 (CD/DAT3)
- net SD2_CLK: now also Card2.5 (CLK)
- net SD2_CMD: now also Card2.2 (CMD)
- net SD2_D0: now also Card2.7 (DAT0)
- net SD2_D1: now also Card2.8 (DAT1)
- net SD2_D2: now also Card2.9 (DAT2)
- net SD2_D3: now also Card2.1 (CD/DAT3)
- net USBA1_DM: now also USB1.2 (D-)
- net USBA1_DP: now also USB1.3 (D+)
- net USBA2_DM: now also USB2.2 (D-)
- net USBA2_DP: now also USB2.3 (D+)
- net USB_DM: now also USB3.A7 (Dn1), USB3.B7 (Dn2)
- net USB_DP: now also USB3.A6 (Dp1), USB3.B6 (Dp2)
- net VBUS: now also IC3.10 (5V), IC4.10 (5V), USB1.1 (VCC), USB2.1 (VCC), USB3.B4A9 (VBUS)
- net at IC4.8 (PMOS): now also Card2.4 (VDD)
- net at IC3.8 (PMOS): now also Card1.4 (VDD)
- net at R10.2: now also USB3.B5 (CC2)
- new net: R23.2, USB3.A5 (CC1)
- no-connect marks 6 -> 8
Other:
- moved on the sheet: C10, C11, C13, C19, TP1, TP2, U1
